File: hw/sch_pcb/VCAI2C02.kicad_pcb (KiCad board)
At the start: 2 copper layers, 70.6 x 30 mm, 43 parts, among them J1 IN 50V(max), J4 BUS I2C, J5 EXT_POWER, J6 ADDR, U1 ADuM3190ARQZ, U2 MCP3423-E/UN

Commit message: update kicad
Other:
- net class Default removed
