File: hw/sch_pcb/VCAI2C02.kicad_sch (KiCad schematic)
At the start: 43 parts

Commit message: update kicad
Parts:
- C10, C4, C9: value (none) -> 100n; footprint (none) -> Capacitor_SMD:C_0805_2012Metric
- C11: value (none) -> 10uF; footprint (none) -> Capacitor_Tantalum_SMD:CP_EIA-3528-21_Kemet-B
- C3, C5, C6: value (none) -> 1u; footprint (none) -> Capacitor_SMD:C_0805_2012Metric
- C7, C8: value (none) -> 10n; footprint (none) -> Capacitor_SMD:C_0805_2012Metric
- D1: value (none) -> MM5Z10VT1G; footprint (none) -> Diode_SMD:D_SOD-523
- D2: value (none) -> +5V -Green; footprint (none) -> Mlab_D:LED_1206
- D3: value (none) -> CDBHM260L-HF; footprint (none) -> Mlab_D:MSB-2
- J1: value (none) -> IN 50V(max); footprint (none) -> Mlab_CON:XT30PW-M
- J4: value (none) -> BUS I2C; footprint (none) -> Mlab_Pin_Headers:Straight_2x05
- J5: value (none) -> EXT_POWER; footprint (none) -> Mlab_Pin_Headers:Straight_2x01
- J6: value (none) -> ADDR; footprint (none) -> Mlab_Pin_Headers:Straight_2x02
- L1: value (none) -> BLM21PG300SN1D; footprint (none) -> Mlab_L:BLM21PG_3Amp
- MH1, MH2, MH3, MH4: value (none) -> MountingHole_Pad; footprint (none) -> Mlab_Mechanical:MountingHole_3mm
- R1, R2, R7, R8: value (none) -> 1M; footprint (none) -> Resistor_SMD:R_0805_2012Metric
- R10, R12, R14, R22, R24: value (none) -> 10k; footprint (none) -> Resistor_SMD:R_0805_2012Metric
- R11: value (none) -> 3k9; footprint (none) -> Resistor_SMD:R_0805_2012Metric
- R13: value (none) -> 330R; footprint (none) -> Resistor_SMD:R_0805_2012Metric
- R15, R16: value (none) -> 180k; footprint (none) -> Resistor_SMD:R_0805_2012Metric
- R17, R18: value (none) -> 33k; footprint (none) -> Resistor_SMD:R_0805_2012Metric
- R3: value (none) -> 50k; footprint (none) -> Resistor_SMD:R_0805_2012Metric
- R4: value (none) -> 40k2; footprint (none) -> Resistor_SMD:R_0805_2012Metric
- R5: value (none) -> 1k5; footprint (none) -> Resistor_SMD:R_0805_2012Metric
- R6: value (none) -> 16k9; footprint (none) -> Resistor_SMD:R_0805_2012Metric
- TR1: value (none) -> L01ZxxxS05; footprint (none) -> Mlab_TR:L01ZxxxS05
- U1: value (none) -> ADuM3190ARQZ; footprint (none) -> Mlab_IO:QSOP-16_3.9x4.9mm_P0.635mm
- U2: value (none) -> MCP3423-E/UN; footprint (none) -> Mlab_IO:MSOP-10_3x3mm_P0.5mm
